File: fabrication/jackboard/USB_distri.kicad_pcb (KiCad board)
At the start: 2 copper layers, 22.5 x 30 mm, 5 parts, among them J1 GSB11111ALF, J2 GSB11111ALF, J3 Power_Input

Commit message: update silkscreen with info on polarity + readme
Other:
- board text added: "5V"
- board text added: "GND"
Changed lines of the file:
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@@
     (effects (font (size 1 1) (thickness 0.15)) (justify mirror))
+  )
+  (gr_text "GND" (at 141.75 69.5) (layer "B.SilkS")
+    (effects (font (size 1 1) (thickness 0.15)) (justify left bottom mirror))
+  )
+  (gr_text "5V" (at 141.75 78.75) (layer "B.SilkS")
+    (effects (font (size 1 1) (thickness 0.15)) (justify left bottom mirror))
   )
   (gr_text "V1.0 BleepSound 2023\n" (at 146 60.3) (layer "B.SilkS")
